Commit message: ros2_ws models test

File: PV1/ros2_ws/src/ball_tracker/urdf/court.urdf (robot description, URDF)
Before this commit: robot volleyball_court, 2 links, 1 joints
Links:
- link court_link: geometry visual box size=18 9 0.1

Commit message: ros2_ws models test

File: PV1/ros2_ws/src/ball_tracker/urdf/court.urdf (robot description, URDF)
Before this commit: robot volleyball_court, 2 links, 1 joints
Links:
- link court_link: geometry visual box size=20 20 20

Commit message: ros2_ws models test

File: PV1/ros2_ws/src/ball_tracker/urdf/court.urdf (robot description, URDF)
Before this commit: robot volleyball_court, 2 links, 1 joints
Links:
- link court_link: geometry visual mesh filename=package://ball_tracker/meshes/model.dae

Commit message: ros2_ws models test

File: PV1/ros2_ws/src/ball_tracker/urdf/court.urdf (robot description, URDF)
Before this commit: robot volleyball_court, 2 links, 1 joints
Links:
- link court_link: geometry visual mesh filename=package://ball_tracker/meshes/Untitled.dae

Commit message: court updates

File: PV1/ros2_ws/src/ball_tracker/urdf/court.urdf (robot description, URDF)
Before this commit: robot volleyball_court, 2 links, 1 joints
Links:
- link court_link: geometry visual mesh filename=package://ball_tracker/meshes/Model.dae

Commit message: court updates

File: PV1/ros2_ws/src/ball_tracker/urdf/court.urdf (robot description, URDF)
Before this commit: robot volleyball_court, 2 links, 1 joints
Links:
- link court_link: geometry visual mesh filename=package://ball_tracker/meshes/untitled.stl
